File: ble_clone.brd (EAGLE design)
At the start: 67.3 x 70.8 mm, 28 parts, among them IC1 PIC24FV16KM202, IC2 3.3 vreg, X1 MCP3208

Commit message: updates
Parts:
- added K1, K2: AQV254R, relay:DIL06
- added LED2: r2, led:LED3MM
- added LED3: r1, led:LED3MM
- added LED4: a0, led:LED3MM
- added LED5: a1, led:LED3MM
- added R10, R11, R5, R6, R7, R8, R9: 470, resistor:0204V
Connections:
- new net N$45: K1.2, R6.2
- new net N$46: K2.2, R7.2
- new net N$47: LED2.A, R8.1
- new net N$48: LED3.A, R9.1
- new net N$51: LED4.A, R10.1
- new net N$52: LED5.A, R11.1
- net N$2: now also R5.2
- net N$24: now also LED4.K
- net N$25: now also LED2.K, R7.1
- net N$26: now also LED3.K, R6.1
- net N$6: now also R5.1
- net N$7: now also LED5.K
- net VDD: now also K1.1, K2.1, R10.2, R11.2, R8.2, R9.2
Routing:
- net N$25: track 36.6 -> 130.3 mm, vias 0 -> 1
- net VDD: track 185.7 -> 257.0 mm, vias 1 -> 0
- net N$14: track 94.5 -> 34.1 mm
- net N$7: track 80.2 -> 135.2 mm
- net N$26: track 45.2 -> 86.4 mm, vias 1 -> 0
- net N$46: track 0.00 -> 38.1 mm
- net N$24: track 48.7 -> 70.6 mm
- net N$13: track 45.3 -> 66.8 mm, vias 2 -> 1
- net GND: track 260.0 -> 240.0 mm
- net N$6: track 9.23 -> 24.9 mm
- net N$11: track 31.4 -> 47.1 mm, vias 1 -> 0
- net N$15: track 23.1 -> 36.2 mm
- net N$45: track 0.00 -> 11.7 mm
- net N$12: track 51.3 -> 60.9 mm, vias 2 -> 3
- net N$48: track 0.00 -> 7.93 mm
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
Commit message: update
Parts:
- added C11: 10uf, resistor:TAP5-45
- added C12, C13, C15: 0.1, resistor:C025-024X044
- added C14: 16uf, resistor:TAP5-45
- added IC3: PIC24FV16KM202, pic24kakl:DIL28-3
- added K3, K4: AQV254R, relay:DIL06
- added R12, R14, R15: 470, resistor:0204V
- added R13: 10k, resistor:0204V
- moved K2 11.4 mm to (50.8, 47.0)
- moved K1 10.2 mm to (39.4, 47.0)
Connections:
- new net N$42: C11.+, C12.1, IC3.20
- new net N$44: K3.2, R14.2
- new net N$49: C15.1, R12.2, R13.1
- new net N$50: IC3.1, R12.1
- new net N$53: K4.2, R15.2
- net GND: now also C11.-, C12.2, C13.2, C14.-, C15.2, IC3.27, IC3.8
- net N$19: now also IC3.15
- net N$20: now also IC3.19
- net N$21: now also IC3.14
- net N$23: now also IC3.23
- net N$24: now also R14.1
- net N$7: now also R15.1
- net VDD: now also C13.1, C14.+, IC3.13, IC3.28, K3.1, K4.1, R13.2
Routing:
- net GND: track 240.0 -> 371.3 mm, vias 1 -> 0
- net N$21: track 14.6 -> 95.8 mm
- net N$20: track 20.8 -> 99.4 mm
- net N$19: track 36.4 -> 113.6 mm
- net VDD: track 257.0 -> 330.7 mm, vias 0 -> 1
- net N$23: track 42.6 -> 115.4 mm, vias 1 -> 0
- net N$3: track 53.7 -> 102.0 mm, vias 0 -> 1
- net N$11: track 47.1 -> 24.5 mm
- net N$13: track 66.8 -> 47.0 mm, vias 1 -> 2
- net N$7: track 135.2 -> 115.5 mm, vias 0 -> 1
- net N$10: track 26.8 -> 43.3 mm
- net N$16: track 71.9 -> 88.0 mm
- net N$24: track 70.6 -> 84.4 mm
- net N$9: track 35.5 -> 49.1 mm
- net N$15: track 36.2 -> 23.4 mm
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Other:
- board size 67.3 x 70.8 mm -> 109.2 x 70.8 mm
