File: ble_clone.brd (EAGLE design)
At the start: 109.2 x 70.8 mm, 53 parts, among them IC1 PIC24FV16KM202, IC2 3.3 vreg, IC3 PIC24FV16KM202, K1 AQV254R, K2 AQV254R, K3 AQV254R, K4 AQV254R, X1 MCP3208

Commit message: updates
Parts:
- added SV7: BT serial, con-lstb:MA06-1
Connections:
- removed net N$4: IC1.6, U$1.P05
- net GND: now also SV7.6
- net N$10: now also SV7.4
- net N$3: now also IC1.6, SV7.1, SV7.2, U$1.P05
- net N$9: now also SV7.3
Routing:
- net N$10: track 43.3 -> 96.9 mm, vias 0 -> 1
- net N$9: track 49.1 -> 95.6 mm, vias 2 -> 4
- net N$7: track 115.5 -> 156.5 mm, vias 1 -> 0
- net N$4: track 34.5 -> 0.00 mm
- net N$14: track 38.4 -> 70.5 mm, vias 2 -> 0
- net VDD: track 330.7 -> 359.1 mm, vias 1 -> 2
- net N$16: track 88.0 -> 69.9 mm
- net N$29: track 16.9 -> 32.3 mm, vias 0 -> 1
- net N$25: track 118.6 -> 133.4 mm, vias 2 -> 1
- net N$31: track 18.3 -> 31.6 mm, vias 1 -> 2
- net N$46: track 48.2 -> 60.1 mm
- net N$3: track 102.0 -> 91.9 mm, vias 1 -> 2
- net N$21: track 95.8 -> 103.1 mm
- net N$12: track 51.1 -> 57.7 mm
- net N$24: track 84.4 -> 78.1 mm
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
Commit message: updates
Routing:
- net GND: track 373.5 -> 0.00 mm
- net VDD: track 359.1 -> 0.00 mm, vias 2 -> 0
- net N$7: track 156.5 -> 0.00 mm
- net N$25: track 133.4 -> 0.00 mm, vias 1 -> 0
- net N$23: track 115.5 -> 0.00 mm, vias 1 -> 0
- net N$19: track 113.6 -> 0.00 mm
- net N$21: track 103.1 -> 0.00 mm
- net N$20: track 99.8 -> 0.00 mm
- net N$10: track 96.9 -> 0.00 mm, vias 1 -> 0
- net N$9: track 95.6 -> 0.00 mm, vias 4 -> 0
- net N$3: track 91.9 -> 0.00 mm, vias 2 -> 0
- net N$26: track 85.1 -> 0.00 mm, vias 1 -> 0
- net N$24: track 78.1 -> 0.00 mm
- net N$14: track 70.5 -> 0.00 mm
- net N$16: track 69.9 -> 0.00 mm
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
Commit message: updates
Routing:
- net GND: track 0.00 -> 373.5 mm
- net VDD: track 0.00 -> 359.1 mm, vias 0 -> 2
- net N$7: track 0.00 -> 156.5 mm
- net N$25: track 0.00 -> 133.4 mm, vias 0 -> 1
- net N$23: track 0.00 -> 115.5 mm, vias 0 -> 1
- net N$19: track 0.00 -> 113.6 mm
- net N$21: track 0.00 -> 103.1 mm
- net N$20: track 0.00 -> 99.8 mm
- net N$10: track 0.00 -> 96.9 mm, vias 0 -> 1
- net N$9: track 0.00 -> 95.6 mm, vias 0 -> 4
- net N$3: track 0.00 -> 91.9 mm, vias 0 -> 2
- net N$26: track 0.00 -> 85.1 mm, vias 0 -> 1
- net N$24: track 0.00 -> 78.1 mm
- net N$14: track 0.00 -> 70.5 mm
- net N$16: track 0.00 -> 69.9 mm
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
Commit message: update code
Parts:
- added CON1: MIKROE_BUS_CONN, mikrobus_lib:MIKROBUS_HOST_CONN
- moved C15 3.81 mm to (83.8, 94.0)
- moved R12 3.81 mm to (88.9, 94.0)
- moved R13 3.81 mm to (88.9, 96.5)
Connections:
- net GND: now also CON1.P$8, CON1.P$9
- net N$1: now also CON1.P$16
- net N$10: now also CON1.P$11, CON1.P$15
- net N$11: now also CON1.P$4
- net N$12: now also CON1.P$5
- net N$13: now also CON1.P$1
- net N$3: now also CON1.P$13, CON1.P$14
- net N$5: now also CON1.P$2
- net N$9: now also CON1.P$12, CON1.P$3
- net VDD: now also CON1.P$7
Routing:
- net N$1: track 18.9 -> 124.7 mm
- net N$9: track 95.6 -> 181.0 mm, vias 4 -> 2
- net N$5: track 20.8 -> 75.3 mm
- net N$3: track 91.9 -> 143.3 mm, vias 2 -> 4
- net N$10: track 96.9 -> 144.4 mm, vias 1 -> 2
- net N$11: track 24.1 -> 65.2 mm, vias 0 -> 1
- net N$7: track 156.5 -> 118.4 mm, vias 0 -> 1
- net GND: track 373.5 -> 407.7 mm, vias 0 -> 1
- net N$14: track 70.5 -> 40.4 mm, vias 0 -> 2
- net N$26: track 85.1 -> 110.0 mm, vias 1 -> 2
- net N$13: track 48.9 -> 67.5 mm, vias 2 -> 1
- net N$46: track 60.1 -> 42.4 mm
- net N$29: track 32.3 -> 16.9 mm, vias 1 -> 0
- net N$31: track 31.6 -> 18.2 mm
- net VDD: track 359.1 -> 345.7 mm, vias 2 -> 0
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Other:
- board size 109.2 x 70.8 mm -> 109.2 x 68.2 mm

Commit message: update
Parts:
- removed C15: 0.1, resistor:C025-024X044
- removed R5: 470, resistor:0204V
- added C16: 0.1, rcl:C0805
- C12, C13: device resistor:C025-024X044 -> rcl:C0805
- R1: value 470 -> 220
- moved C12 106.4 mm to (20.3, 3.81)
- moved SV7 94.1 mm to (59.7, 5.08), turned to 0 degrees
- moved PAD2 87.7 mm to (5.08, 2.54)
- moved PAD1 86.7 mm to (14.0, 2.54)
- moved C11 85.9 mm to (27.9, 35.6)
- moved C13 84.6 mm to (25.4, 3.81), turned to 0 degrees
- moved L1 75.2 mm to (20.3, 21.6), turned to 90 degrees
- moved SV3 70.1 mm to (77.5, 5.08), turned to 180 degrees
- moved IC2 66.9 mm to (10.2, 11.4)
- moved R12 65.1 mm to (38.1, 53.3), turned to 0 degrees
- moved C14 64.4 mm to (35.6, 35.6), turned to 0 degrees
- moved R13 64.3 mm to (38.1, 57.1), turned to 0 degrees
- moved C6 63.8 mm to (12.7, 35.6)
- moved SV4 59.2 mm to (8.89, 29.2), turned to 0 degrees
- moved LED1 57.8 mm to (3.81, 35.6)
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Connections:
- new net N$4: CON1.P$14, IC1.16, SV7.1, U$1.P06
- net GND: now also C16.2; no longer C15.2
- net N$2: no longer R5.2
- net N$3: no longer CON1.P$14, IC1.16, SV7.1, U$1.P06
- net N$49: now also C16.1; no longer C15.1
- net N$6: no longer R5.1
Routing:
- net N$4: track 0.00 -> 211.6 mm, vias 0 -> 3
- net N$42: track 6.94 -> 116.3 mm, vias 0 -> 1
- net N$18: track 35.4 -> 122.6 mm
- net N$23: track 127.2 -> 195.4 mm, vias 1 -> 0
- net N$44: track 3.89 -> 69.9 mm
- net N$50: track 5.43 -> 58.9 mm
- net N$19: track 112.4 -> 165.6 mm, vias 1 -> 0
- net N$16: track 69.1 -> 121.2 mm
- net N$3: track 143.3 -> 195.0 mm, vias 4 -> 3
- net N$49: track 6.37 -> 56.9 mm
- net N$24: track 80.7 -> 122.4 mm, vias 0 -> 1
- net N$27: track 5.08 -> 46.0 mm
- net N$13: track 67.5 -> 107.4 mm, vias 1 -> 2
- net N$7: track 118.4 -> 157.6 mm, vias 1 -> 0
- net VDD: track 345.7 -> 383.4 mm, vias 0 -> 3
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Other:
- board size 109.2 x 68.2 mm -> 100 x 80 mm
