File: ble_clone.sch (EAGLE design)
At the start: 24 parts, among them IC1 PIC24FV16KM202, IC2 3.3 vreg

Commit message: updates
Parts:
- added C10: 0.1, resistor:C-US025-024X044
- added R4: 50, resistor:R-US_0204/2V
- added SV6: analog input, con-lstb:MA10-1
- added X1: MCP3208, Microchip:21298EDIP
Connections:
- new net N$34: SV6.2, X1.CH7
- new net N$35: SV6.3, X1.CH6
- new net N$36: SV6.4, X1.CH5
- new net N$37: SV6.5, X1.CH4
- new net N$38: SV6.6, X1.CH3
- new net N$39: SV6.7, X1.CH2
- new net N$40: SV6.8, X1.CH1
- new net N$41: SV6.9, X1.CH0
- new net N$43: R4.1, SV6.10
- net GND: now also C10.2, SV6.1, X1.AGND, X1.DGND
- net N$16: now also C10.1, R4.2, X1.VDD, X1.VREF
- net N$18: now also X1.!CS
- net N$19: now also X1.DOUT
- net N$20: now also X1.DIN
- net N$21: now also X1.CLK
Other:
- moved on the sheet: SV3

Commit message: updates
Parts:
- added K1, K2: AQV254R, relay:AQV254R
- added LED2: r2, led:LED3MM
- added LED3: r1, led:LED3MM
- added LED4: a0, led:LED3MM
- added LED5: a1, led:LED3MM
- added R10, R11, R5, R6, R7, R8, R9: 470, resistor:R-US_0204/2V
Connections:
- new net N$45: K1.K, R6.2
- new net N$46: K2.K, R7.2
- new net N$47: LED2.A, R8.1
- new net N$48: LED3.A, R9.1
- new net N$51: LED4.A, R10.1
- new net N$52: LED5.A, R11.1
- net N$2: now also R5.2
- net N$24: now also LED4.C
- net N$25: now also LED2.C, R7.1
- net N$26: now also LED3.C, R6.1
- net N$6: now also R5.1
- net N$7: now also LED5.C
- net VDD: now also K1.A, K2.A, R10.2, R11.2, R8.2, R9.2
Changed lines of the file:
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@@
 <part name="R4" library="resistor" deviceset="R-US_" device="0204/2V" value="50"/>
 <part name="SUPPLY19" library="supply2" deviceset="GND" device=""/>
+<part name="K1" library="relay" deviceset="AQV254R" device=""/>
+<part name="K2" library="relay" deviceset="AQV254R" device=""/>
+<part name="VDD6" library="supply1" deviceset="VDD" device=""/>
+<part name="VDD7" library="supply1" deviceset="VDD" device=""/>
+<part name="R5" library="resistor" deviceset="R-US_" device="0204/2V" value="470"/>
+<part name="R6" library="resistor" deviceset="R-US_" device="0204/2V" value="470"/>
+<part name="R7" library="resistor" deviceset="R-US_" device="0204/2V" value="470"/>
+<part name="LED2" library="led" deviceset="LED" device="3MM" value="r2"/>
+<part name="LED3" library="led" deviceset="LED" device="3MM" value="r1"/>
+<part name="R8" library="resistor" deviceset="R-US_" device="0204/2V" value="470"/>
+<part name="R9" library="resistor" deviceset="R-US_" device="0204/2V" value="470"/>
+<part name="LED4" library="led" deviceset="LED" device="3MM" value="a0"/>
+<part name="LED5" library="led" deviceset="LED" device="3MM" value="a1"/>
+<part name="R10" library="resistor" deviceset="R-US_" device="0204/2V" value="470"/>
+<part name="R11" library="resistor" deviceset="R-US_" device="0204/2V" value="470"/>
+<part name="VDD8" library="supply1" deviceset="VDD" device=""/>
 </parts>
 <sheets>
@@
 <instance part="R4" gate="G$1" x="-45.72" y="-43.18" rot="R180"/>
 <instance part="SUPPLY19" gate="GND" x="7.62" y="-45.72"/>
+<instance part="K1" gate="G$1" x="205.74" y="-15.24"/>
+<instance part="K2" gate="G$1" x="205.74" y="-43.18"/>
+<instance part="VDD6" gate="G$1" x="190.5" y="-7.62"/>
+<instance part="VDD7" gate="G$1" x="190.5" y="-35.56"/>
+<instance part="R5" gate="G$1" x="50.8" y="71.12"/>
+<instance part="R6" gate="G$1" x="190.5" y="-20.32"/>
+<instance part="R7" gate="G$1" x="190.5" y="-48.26"/>
+<instance part="LED2" gate="G$1" x="182.88" y="-43.18"/>
+<instance part="LED3" gate="G$1" x="182.88" y="-15.24"/>
+<instance part="R8" gate="G$1" x="182.88" y="-35.56" rot="R90"/>
+<instance part="R9" gate="G$1" x="182.88" y="-7.62" rot="R90"/>
+<instance part="LED4" gate="G$1" x="154.94" y="-40.64"/>
+<instance part="LED5" gate="G$1" x="165.1" y="-40.64"/>
+<instance part="R10" gate="G$1" x="154.94" y="-33.02" rot="R90"/>
+<instance part="R11" gate="G$1" x="165.1" y="-33.02" rot="R90"/>
+<instance part="VDD8" gate="G$1" x="160.02" y="-25.4"/>
 </instances>
 <busses>
@@
 <junction x="149.86" y="-7.62"/>
 </segment>
+<segment>
+<pinref part="K1" gate="G$1" pin="A"/>
+<wire x1="190.5" y1="-10.16" x2="195.58" y2="-10.16" width="0.1524" layer="91"/>
+<pinref part="VDD6" gate="G$1" pin="VDD"/>
+<pinref part="R9" gate="G$1" pin="2"/>
+<wire x1="182.88" y1="-2.54" x2="195.58" y2="-2.54" width="0.1524" layer="91"/>
+<wire x1="195.58" y1="-2.54" x2="195.58" y2="-10.16" width="0.1524" layer="91"/>
+<junction x="195.58" y="-10.16"/>
+</segment>
+<segment>
+<pinref part="K2" gate="G$1" pin="A"/>
+<wire x1="190.5" y1="-38.1" x2="195.58" y2="-38.1" width="0.1524" layer="91"/>
+<pinref part="VDD7" gate="G$1" pin="VDD"/>
+<pinref part="R8" gate="G$1" pin="2"/>
+<wire x1="182.88" y1="-30.48" x2="195.58" y2="-30.48" width="0.1524" layer="91"/>
+<wire x1="195.58" y1="-30.48" x2="195.58" y2="-38.1" width="0.1524" layer="91"/>
+<junction x="195.58" y="-38.1"/>
+</segment>
+<segment>
+<pinref part="R10" gate="G$1" pin="2"/>
+<pinref part="R11" gate="G$1" pin="2"/>
+<wire x1="154.94" y1="-27.94" x2="160.02" y2="-27.94" width="0.1524" layer="91"/>
+<pinref part="VDD8" gate="G$1" pin="VDD"/>
+<wire x1="160.02" y1="-27.94" x2="165.1" y2="-27.94" width="0.1524" layer="91"/>
+<junction x="160.02" y="-27.94"/>
+</segment>
 </net>
 <net name="N$2" class="0">
@@
 <pinref part="SV2" gate="1" pin="1"/>
 <wire x1="83.82" y1="83.82" x2="83.82" y2="86.36" width="0.1524" layer="91"/>
+<pinref part="R5" gate="G$1" pin="2"/>
 </segment>
 </net>
@@
 <pinref part="IC1" gate="G$1" pin="RA5/!MCLR"/>
 <wire x1="35.56" y1="35.56" x2="40.64" y2="35.56" width="0.1524" layer="91"/>
+<pinref part="R5" gate="G$1" pin="1"/>
+<junction x="45.72" y="71.12"/>
 </segment>
 </net>
@@
 <junction x="124.46" y="45.72"/>
 <junction x="162.56" y="-7.62"/>
+<pinref part="LED5" gate="G$1" pin="C"/>
+<wire x1="165.1" y1="-45.72" x2="165.1" y2="-48.26" width="0.1524" layer="91"/>
+<wire x1="165.1" y1="-48.26" x2="172.72" y2="-48.26" width="0.1524" layer="91"/>
+<wire x1="172.72" y1="-48.26" x2="172.72" y2="-7.62" width="0.1524" layer="91"/>
+<wire x1="172.72" y1="-7.62" x2="162.56" y2="-7.62" width="0.1524" layer="91"/>
 </segment>
 </net>
@@
 <wire x1="152.4" y1="30.48" x2="160.02" y2="30.48" width="0.1524" layer="91"/>
 <pinref part="SV4" gate="1" pin="2"/>
-<wire x1="160.02" y1="30.48" x2="160.02" y2="-7.62" width="0.1524" layer="91"/>
+<wire x1="160.02" y1="30.48" x2="160.02" y2="0" width="0.1524" layer="91"/>
 <junction x="160.02" y="-7.62"/>
+<pinref part="LED4" gate="G$1" pin="C"/>
+<wire x1="160.02" y1="0" x2="160.02" y2="-7.62" width="0.1524" layer="91"/>
+<wire x1="154.94" y1="-45.72" x2="154.94" y2="-53.34" width="0.1524" layer="91"/>
+<wire x1="154.94" y1="-53.34" x2="175.26" y2="-53.34" width="0.1524" layer="91"/>
+<wire x1="175.26" y1="-53.34" x2="175.26" y2="0" width="0.1524" layer="91"/>
+<wire x1="175.26" y1="0" x2="160.02" y2="0" width="0.1524" layer="91"/>
+<junction x="160.02" y="0"/>
 </segment>
 </net>
@@
 <pinref part="IC1" gate="G$1" pin="AN12/INT2/!SS2!/CN14/RB12"/>
 <wire x1="116.84" y1="22.86" x2="157.48" y2="22.86" width="0.1524" layer="91"/>
-<wire x1="157.48" y1="22.86" x2="157.48" y2="-7.62" width="0.1524" layer="91"/>
+<wire x1="157.48" y1="22.86" x2="157.48" y2="-2.54" width="0.1524" layer="91"/>
 <pinref part="SV4" gate="1" pin="3"/>
 <junction x="157.48" y="-7.62"/>
+<wire x1="157.48" y1="-2.54" x2="157.48" y2="-7.62" width="0.1524" layer="91"/>
 <wire x1="157.48" y1="-7.62" x2="157.48" y2="-10.16" width="0.1524" layer="91"/>
+<wire x1="157.48" y1="-2.54" x2="177.8" y2="-2.54" width="0.1524" layer="91"/>
+<wire x1="177.8" y1="-2.54" x2="177.8" y2="-48.26" width="0.1524" layer="91"/>
+<pinref part="R7" gate="G$1" pin="1"/>
+<wire x1="177.8" y1="-48.26" x2="182.88" y2="-48.26" width="0.1524" layer="91"/>
+<junction x="157.48" y="-2.54"/>
+<pinref part="LED2" gate="G$1" pin="C"/>
+<wire x1="182.88" y1="-48.26" x2="185.42" y2="-48.26" width="0.1524" layer="91"/>
+<junction x="182.88" y="-48.26"/>
 </segment>
 </net>
@@
 <wire x1="116.84" y1="20.32" x2="154.94" y2="20.32" width="0.1524" layer="91"/>
 <pinref part="SV4" gate="1" pin="4"/>
-<wire x1="154.94" y1="20.32" x2="154.94" y2="-7.62" width="0.1524" layer="91"/>
+<wire x1="154.94" y1="20.32" x2="154.94" y2="-5.08" width="0.1524" layer="91"/>
 <junction x="154.94" y="-7.62"/>
+<wire x1="154.94" y1="-5.08" x2="154.94" y2="-7.62" width="0.1524" layer="91"/>
+<wire x1="154.94" y1="-5.08" x2="180.34" y2="-5.08" width="0.1524" layer="91"/>
+<wire x1="180.34" y1="-5.08" x2="180.34" y2="-20.32" width="0.1524" layer="91"/>
+<pinref part="R6" gate="G$1" pin="1"/>
+<wire x1="180.34" y1="-20.32" x2="182.88" y2="-20.32" width="0.1524" layer="91"/>
+<junction x="154.94" y="-5.08"/>
+<pinref part="LED3" gate="G$1" pin="C"/>
+<wire x1="182.88" y1="-20.32" x2="185.42" y2="-20.32" width="0.1524" layer="91"/>
+<junction x="182.88" y="-20.32"/>
 </segment>
 </net>
@@
 </segment>
 </net>
+<net name="N$45" class="0">
+<segment>
+<pinref part="K1" gate="G$1" pin="K"/>
+<pinref part="R6" gate="G$1" pin="2"/>
+</segment>
+</net>
+<net name="N$46" class="0">
+<segment>
+<pinref part="K2" gate="G$1" pin="K"/>
+<pinref part="R7" gate="G$1" pin="2"/>
+</segment>
+</net>
+<net name="N$47" class="0">
+<segment>
+<pinref part="LED2" gate="G$1" pin="A"/>
+<pinref part="R8" gate="G$1" pin="1"/>
+</segment>
+</net>
+<net name="N$48" class="0">
+<segment>
+<pinref part="LED3" gate="G$1" pin="A"/>
+<pinref part="R9" gate="G$1" pin="1"/>
+</segment>
+</net>
+<net name="N$51" class="0">
+<segment>
+<pinref part="LED4" gate="G$1" pin="A"/>
+<pinref part="R10" gate="G$1" pin="1"/>
+</segment>
+</net>
+<net name="N$52" class="0">
+<segment>
+<pinref part="LED5" gate="G$1" pin="A"/>
+<pinref part="R11" gate="G$1" pin="1"/>
+</segment>
+</net>

Commit message: update
Parts:
- added C11: 10uf, resistor:CPOL-USTAP5-45
- added C12, C13, C15: 0.1, resistor:C-US025-024X044
- added C14: 16uf, resistor:CPOL-USTAP5-45
- added IC3: PIC24FV16KM202, pic24kakl:PIC24FVXXKA302-SP
- added K3, K4: AQV254R, relay:AQV254R
- added R12, R14, R15: 470, resistor:R-US_0204/2V
- added R13: 10k, resistor:R-US_0204/2V
Connections:
- new net N$42: C11.+, C12.1, IC3.VCAP
- new net N$44: K3.K, R14.2
- new net N$49: C15.1, R12.2, R13.1
- new net N$50: IC3.RA5/!MCLR, R12.1
- new net N$53: K4.K, R15.2
- net GND: now also C11.-, C12.2, C13.2, C14.-, C15.2, IC3.GND@1, IC3.GND@2
- net N$19: now also IC3.PGEC3/ASCL1/SDO2/CN24/RB6
- net N$20: now also IC3.RA7/CN9/SDI2
- net N$21: now also IC3.PGED3/ASDA1/SCK2/CN27/RB5
- net N$23: now also IC3.AN12/INT2/!SS2!/CN14/RB12
- net N$24: now also R14.1
- net N$7: now also R15.1
- net VDD: now also C13.1, C14.+, IC3.VDD@1, IC3.VDD@2, K3.A, K4.A, R13.2

Commit message: update
Other:
- note added: "seperate pin"
Changed lines of the file:
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@@
 <text x="213.36" y="76.2" size="1.778" layer="91">conn</text>
 <text x="233.68" y="76.2" size="1.778" layer="91">wake</text>
+<text x="-10.16" y="25.4" size="1.778" layer="91">seperate pin</text>
 </plain>
 <instances>
