File: ble_clone.sch (EAGLE design)
At the start: 53 parts, among them IC1 PIC24FV16KM202, IC2 3.3 vreg, IC3 PIC24FV16KM202, K1 AQV254R, K2 AQV254R, K3 AQV254R, K4 AQV254R, X1 MCP3208

Commit message: updates
Parts:
- added SV7: BT serial, con-lstb:MA06-1
Connections:
- removed net N$4: IC1.AN4/SDA2/U1RX/CN6/RB2, U$1.5-TX
- net GND: now also SV7.6
- net N$10: now also SV7.4
- net N$3: now also IC1.AN4/SDA2/U1RX/CN6/RB2, SV7.1, SV7.2, U$1.5-TX
- net N$9: now also SV7.3

Commit message: updates
Changed lines of the file:
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@@
 <net name="N$3" class="0">
 <segment>
-<pinref part="U$1" gate="G$1" pin="6-RX"/>
-<wire x1="152.4" y1="68.58" x2="129.54" y2="68.58" width="0.1524" layer="91"/>
-<wire x1="129.54" y1="68.58" x2="129.54" y2="40.64" width="0.1524" layer="91"/>
-<pinref part="IC1" gate="G$1" pin="INT0/U1TX/CN23/RB7"/>
-<wire x1="129.54" y1="40.64" x2="129.54" y2="35.56" width="0.1524" layer="91"/>
-<wire x1="129.54" y1="35.56" x2="116.84" y2="35.56" width="0.1524" layer="91"/>
-<wire x1="129.54" y1="40.64" x2="149.86" y2="40.64" width="0.1524" layer="91"/>
-<wire x1="149.86" y1="40.64" x2="149.86" y2="27.94" width="0.1524" layer="91"/>
-<wire x1="149.86" y1="27.94" x2="149.86" y2="17.78" width="0.1524" layer="91"/>
 <wire x1="149.86" y1="17.78" x2="195.58" y2="17.78" width="0.1524" layer="91"/>
 <wire x1="195.58" y1="17.78" x2="195.58" y2="43.18" width="0.1524" layer="91"/>
 <wire x1="195.58" y1="43.18" x2="220.98" y2="43.18" width="0.1524" layer="91"/>
-<junction x="129.54" y="40.64"/>
 <pinref part="U$1" gate="G$1" pin="5-TX"/>
 <wire x1="220.98" y1="43.18" x2="223.52" y2="43.18" width="0.1524" layer="91"/>
@@
 <wire x1="127" y1="48.26" x2="116.84" y2="48.26" width="0.1524" layer="91"/>
 <wire x1="127" y1="48.26" x2="149.86" y2="48.26" width="0.1524" layer="91"/>
-<wire x1="149.86" y1="48.26" x2="149.86" y2="27.94" width="0.1524" layer="91"/>
+<wire x1="149.86" y1="48.26" x2="149.86" y2="40.64" width="0.1524" layer="91"/>
+<junction x="127" y="48.26"/>
+<pinref part="SV7" gate="1" pin="2"/>
+<junction x="220.98" y="43.18"/>
+<pinref part="IC1" gate="G$1" pin="INT0/U1TX/CN23/RB7"/>
+<pinref part="U$1" gate="G$1" pin="6-RX"/>
+<wire x1="149.86" y1="40.64" x2="149.86" y2="17.78" width="0.1524" layer="91"/>
+<wire x1="152.4" y1="68.58" x2="129.54" y2="68.58" width="0.1524" layer="91"/>
+<wire x1="129.54" y1="68.58" x2="129.54" y2="40.64" width="0.1524" layer="91"/>
+<wire x1="129.54" y1="40.64" x2="129.54" y2="35.56" width="0.1524" layer="91"/>
+<wire x1="129.54" y1="35.56" x2="116.84" y2="35.56" width="0.1524" layer="91"/>
+<pinref part="SV7" gate="1" pin="1"/>
+<wire x1="129.54" y1="40.64" x2="144.78" y2="40.64" width="0.1524" layer="91"/>
+<wire x1="149.86" y1="40.64" x2="149.86" y2="27.94" width="0.1524" layer="91"/>
 <wire x1="149.86" y1="27.94" x2="193.04" y2="27.94" width="0.1524" layer="91"/>
 <wire x1="193.04" y1="27.94" x2="193.04" y2="45.72" width="0.1524" layer="91"/>
-<pinref part="SV7" gate="1" pin="1"/>
 <wire x1="193.04" y1="45.72" x2="220.98" y2="45.72" width="0.1524" layer="91"/>
-<junction x="127" y="48.26"/>
-<junction x="149.86" y="27.94"/>
 <junction x="220.98" y="45.72"/>
-<pinref part="SV7" gate="1" pin="2"/>
-<junction x="220.98" y="43.18"/>
+<wire x1="144.78" y1="40.64" x2="144.78" y2="27.94" width="0.1524" layer="91"/>
+<wire x1="144.78" y1="27.94" x2="149.86" y2="27.94" width="0.1524" layer="91"/>
+<junction x="129.54" y="40.64"/>
+<junction x="149.86" y="40.64"/>
 </segment>
 </net>

Commit message: update code
Parts:
- added CON1: MIKROE_BUS_CONN, mikrobus_lib:MIKROE_BUS_CONN
Connections:
- net GND: now also CON1.GND1, CON1.GND2
- net N$1: now also CON1.PWM
- net N$10: now also CON1.INT, CON1.SDA
- net N$11: now also CON1.SCK
- net N$12: now also CON1.MISO
- net N$13: now also CON1.AN
- net N$3: now also CON1.RX, CON1.TX
- net N$5: now also CON1.RST
- net N$9: now also CON1.CS, CON1.SCL
- net VDD: now also CON1.3V3
Other:
- note added: "RTS 4871 4020 3 12 CTS 15 11"

Commit message: update
Parts:
- removed C15: 0.1, resistor:C-US025-024X044
- removed R5: 470, resistor:R-US_0204/2V
- added C16: 0.1, rcl:C-USC0805
- C12, C13: device resistor:C-US025-024X044 -> rcl:C-USC0805
- R1: value 470 -> 220
Connections:
- new net N$4: CON1.RX, IC1.INT0/U1TX/CN23/RB7, SV7.1, U$1.6-RX
- net GND: now also C16.2; no longer C15.2
- net N$2: no longer R5.2
- net N$3: no longer CON1.RX, IC1.INT0/U1TX/CN23/RB7, SV7.1, U$1.6-RX
- net N$49: now also C16.1; no longer C15.1
- net N$6: no longer R5.1
Other:
- moved on the sheet: C7, R1, R13
